File: Eagle/stavebnice03_base/base3-5pin-interface-SDA-SCL-Switch-on-output-posunute-konektory-posunuty-vstup.sch (EAGLE design)
At the start: 16 parts

Commit message: minor changes
Connections:
- removed net N$16: U$1.RC3, U$9.3
- new net N$3: U$1.RC3, U$9.2
- net N$17: now also U$9.3; no longer U$9.2
Changed lines of the file:
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@@
 <segment>
 <pinref part="U$1" gate="G$1" pin="RC4"/>
-<wire x1="121.92" y1="73.66" x2="124.46" y2="73.66" width="0.1524" layer="91"/>
-<wire x1="121.92" y1="73.66" x2="121.92" y2="43.18" width="0.1524" layer="91"/>
-<pinref part="U$9" gate="G$1" pin="2"/>
+<pinref part="U$9" gate="G$1" pin="3"/>
+<wire x1="124.46" y1="73.66" x2="116.84" y2="73.66" width="0.1524" layer="91"/>
+<wire x1="116.84" y1="73.66" x2="116.84" y2="43.18" width="0.1524" layer="91"/>
 </segment>
 </net>
@@
 <wire x1="124.46" y1="78.74" x2="111.76" y2="78.74" width="0.1524" layer="91"/>
 <wire x1="111.76" y1="78.74" x2="111.76" y2="43.18" width="0.1524" layer="91"/>
-</segment>
-</net>
-<net name="N$16" class="0">
-<segment>
-<pinref part="U$1" gate="G$1" pin="RC3"/>
-<wire x1="124.46" y1="68.58" x2="116.84" y2="68.58" width="0.1524" layer="91"/>
-<wire x1="116.84" y1="68.58" x2="116.84" y2="43.18" width="0.1524" layer="91"/>
-<pinref part="U$9" gate="G$1" pin="3"/>
 </segment>
 </net>
@@
 </segment>
 </net>
+<net name="N$3" class="0">
+<segment>
+<pinref part="U$1" gate="G$1" pin="RC3"/>
+<pinref part="U$9" gate="G$1" pin="2"/>
+<wire x1="124.46" y1="68.58" x2="121.92" y2="68.58" width="0.1524" layer="91"/>
+<wire x1="121.92" y1="68.58" x2="121.92" y2="43.18" width="0.1524" layer="91"/>
+</segment>
+</net>
