File: Eagle/stavebnice03/misc/AAA_third_source.brd (EAGLE design)
At the start: 9 parts

Commit message: I did an order in Eagle files
Parts:
- added R3, TERMISTOR: 10k, resistor:R0603
- added U$2, U$3: AAA_THIRD, !stavebnice03:AAA_THIRD
- R1, R2: value 4k7 -> 2k2
- moved R2 3.04 mm to (14.4, 11.4), turned to 180 degrees
- moved R1 2.88 mm to (14.4, 9.80), turned to 180 degrees
- moved C2 2.02 mm to (8.90, 4.90)
- moved U$7 1.99 mm to (11.5, 12.6)
- moved U$6 1.99 mm to (11.5, 8.40)
- moved U$1 1.97 mm to (6.90, 10.0)
- moved C5 1.91 mm to (11.5, 4.90)
- moved C3 1.55 mm to (12.4, 14.7), turned to 0 degrees
- moved U$5 0.30 mm to (22.2, 10.5)
Connections:
- new net N$2: U$2.P$2, U$3.P$1
- new net N$3: R3.2, TERMISTOR.2, U$1.8
- net GND: now also R3.1, U$3.P$2
- net VCC: now also TERMISTOR.1, U$2.P$1
Routing:
- net GND: track 52.3 -> 73.1 mm, vias 4 -> 9
- net VCC: track 25.3 -> 42.4 mm, vias 4 -> 2
- net N$2: track 0.00 -> 13.1 mm
- net N$3: track 0.00 -> 9.12 mm, vias 0 -> 1
- net N$7: track 23.9 -> 19.4 mm
- net N$6: track 10.3 -> 14.0 mm
- net N$10: track 9.65 -> 11.2 mm
- net N$4: track 7.42 -> 6.59 mm
- added copper zone on layer 1, net GND
Other:
- board text added: "AAA source"
- board text removed: "5 pins - v2"

Commit message: just element moving
Parts:
- moved U$2 1.70 mm to (15.2, 13.9)
- moved U$3 0.71 mm to (5.00, 9.20)
Routing:
- net GND: track 73.1 -> 69.7 mm, vias 9 -> 3
- net N$2: track 13.1 -> 12.1 mm
- net VCC: track 42.4 -> 41.9 mm
Changed lines of the file:
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@@
 <layer number="97" name="Info" color="7" fill="1" visible="no" active="no"/>
 <layer number="98" name="Guide" color="6" fill="1" visible="no" active="no"/>
+<layer number="99" name="SpiceOrder" color="5" fill="1" visible="no" active="no"/>
 <layer number="116" name="centerDrill" color="7" fill="1" visible="yes" active="yes"/>
 </layers>
@@
 <circle x="8.8" y="15.7" radius="0.275" width="0.15" layer="116"/>
 <circle x="8.9" y="10.5" radius="0.275" width="0.15" layer="116"/>
-<circle x="0.8" y="14.6" radius="0.275" width="0.15" layer="116"/>
-<circle x="0.8" y="13.1" radius="0.275" width="0.15" layer="116"/>
-<circle x="0.8" y="11.6" radius="0.275" width="0.15" layer="116"/>
-<circle x="12.3" y="1.7" radius="0.275" width="0.15" layer="116"/>
-<circle x="13.8" y="1.7" radius="0.275" width="0.15" layer="116"/>
-<circle x="15.3" y="1.7" radius="0.275" width="0.15" layer="116"/>
 <circle x="10.1" y="15" radius="0.275" width="0.15" layer="116"/>
 <circle x="10" y="6.7" radius="0.275" width="0.15" layer="116"/>
@@
 <element name="U$7" library="!stavebnice03" package="SC70-6L" value="NC7SB3157P6X" x="11.5" y="12.6" rot="MR0"/>
 <element name="C5" library="resistor" package="C0603" value="100nF" x="11.5" y="4.9" rot="MR90"/>
-<element name="U$2" library="!stavebnice03" package="AAA_THIRD" value="AAA_THIRD" x="15.3" y="12.2" rot="R90"/>
-<element name="U$3" library="!stavebnice03" package="AAA_THIRD" value="AAA_THIRD" x="5.1" y="8.5" rot="R270"/>
+<element name="U$2" library="!stavebnice03" package="AAA_THIRD" value="AAA_THIRD" x="15.2" y="13.9" rot="R90"/>
+<element name="U$3" library="!stavebnice03" package="AAA_THIRD" value="AAA_THIRD" x="5" y="9.2" rot="R270"/>
 <element name="TERMISTOR" library="resistor" package="R0603" value="10k" x="10.1" y="12.4" rot="R90"/>
 <element name="R3" library="resistor" package="R0603" value="10k" x="4.6" y="15" rot="MR270"/>
@@
 <wire x1="18.14" y1="17.1" x2="13.2" y2="17.1" width="0.357" layer="16"/>
 <wire x1="13.2" y1="17.1" x2="11.1" y2="17.1" width="0.357" layer="16"/>
-<wire x1="5.1" y1="4" x2="8.9" y2="8" width="0.357" layer="1"/>
-<wire x1="8.9" y1="8" x2="8.9" y2="10.5" width="0.357" layer="1"/>
 <wire x1="8.9" y1="10.5" x2="8.8" y2="10.7" width="0.357" layer="1"/>
 <wire x1="8.8" y1="10.7" x2="8.8" y2="15.7" width="0.357" layer="1"/>
@@
 <vertex x="21" y="0"/>
 </polygon>
-<via x="0.8" y="14.6" extent="1-16" drill="0.6"/>
-<via x="0.8" y="13.1" extent="1-16" drill="0.6"/>
-<via x="0.8" y="11.6" extent="1-16" drill="0.6"/>
-<via x="12.3" y="1.7" extent="1-16" drill="0.6"/>
-<via x="13.8" y="1.7" extent="1-16" drill="0.6"/>
-<via x="15.3" y="1.7" extent="1-16" drill="0.6"/>
 <contactref element="R3" pad="1"/>
 <wire x1="4.3" y1="16" x2="2.2" y2="13.9" width="0.3556" layer="16"/>
@@
 <wire x1="13.25" y1="17.05" x2="13.2" y2="17.1" width="0.3556" layer="16"/>
 <wire x1="8.9" y1="4.05" x2="11.5" y2="4.05" width="0.3556" layer="16"/>
+<wire x1="5" y1="2.2" x2="7.05" y2="2.2" width="0.4064" layer="16"/>
+<wire x1="7.05" y1="2.2" x2="8.9" y2="4.05" width="0.4064" layer="16"/>
 </signal>
 <signal name="VCC">
@@
 </polygon>
 <contactref element="U$2" pad="P$1"/>
-<wire x1="15.3" y1="7.7" x2="15.75" y2="7.75" width="0.357" layer="1"/>
 <wire x1="11.5" y1="7.55" x2="11.4875" y2="6.8125" width="0.357" layer="16"/>
 <wire x1="11.4875" y1="6.8125" x2="11.5" y2="6.8" width="0.357" layer="16"/>
@@
 <via x="10" y="6.7" extent="1-16" drill="0.6"/>
 <wire x1="10" y1="6.7" x2="14.7" y2="6.7" width="0.357" layer="1"/>
-<wire x1="14.7" y1="6.7" x2="15.3" y2="7.7" width="0.357" layer="1"/>
 <wire x1="11.5" y1="13.45" x2="11.4875" y2="15.9125" width="0.357" layer="16"/>
 <wire x1="11.4875" y1="15.9125" x2="11.5" y2="16" width="0.357" layer="16"/>
@@
 <wire x1="11.5" y1="16" x2="11.5" y2="12" width="0.357" layer="1"/>
 <wire x1="11.5" y1="12" x2="15.2" y2="8.3" width="0.357" layer="1"/>
-<wire x1="15.2" y1="8.3" x2="15.75" y2="7.75" width="0.357" layer="1"/>
 <wire x1="19.66" y1="10.5" x2="17.4" y2="10.5" width="1.016" layer="1"/>
 <wire x1="17.4" y1="10.5" x2="15.2" y2="8.3" width="0.357" layer="1"/>
@@
 <wire x1="11.5" y1="12" x2="10.55" y2="12" width="0.3556" layer="1"/>
 <wire x1="10.55" y1="12" x2="10.1" y2="11.55" width="0.3556" layer="1"/>
+<wire x1="15.2" y1="8.3" x2="15.2" y2="7.2" width="0.4064" layer="1"/>
+<wire x1="15.2" y1="7.2" x2="14.7" y2="6.7" width="0.4064" layer="1"/>
+<wire x1="15.2" y1="7.2" x2="15.2" y2="6.9" width="0" layer="19" extent="1-16"/>
 </signal>
 <signal name="N$19">
@@
 <contactref element="U$2" pad="P$2"/>
 <contactref element="U$3" pad="P$1"/>
-<wire x1="15" y1="17.4" x2="15.3" y2="16.7" width="0.357" layer="1"/>
-<wire x1="15" y1="17.4" x2="8.5" y2="17.4" width="1.016" layer="1"/>
-<wire x1="8.5" y1="17.4" x2="5" y2="13.9" width="1.016" layer="1"/>
-<wire x1="5" y1="13.9" x2="5.1" y2="13" width="0.3556" layer="1"/>
+<wire x1="15.2" y1="20.9" x2="9.7" y2="20.9" width="0.4064" layer="16"/>
+<wire x1="9.7" y1="20.9" x2="5" y2="16.2" width="0.4064" layer="16"/>
 </signal>
 <signal name="N$3">
