File: Eagle/stavebnice03/misc/AAA_third_source.sch (EAGLE design)
At the start: 16 parts

Commit message: I did an order in Eagle files
Parts:
- removed C1, C4: 100nF, resistor:C-EUC0603
- removed U$4: JUMPER5M-90, !stavebnice03:JUMPER5M-90
- removed U$8: JUMPER6M, !stavebnice03:JUMPER6M
- removed U$9: JUMPER4M, !stavebnice03:JUMPER4M
- added R3, TERMISTOR: 10k, resistor:R-EU_R0603
- R1, R2: value 4k7 -> 2k2; device resistor:R-EU_M0805 -> resistor:R-EU_R0603
- U$2, U$3: value NC7SB3157P6X -> AAA_THIRD; device !stavebnice03:NC7SB3157P6X -> !stavebnice03:AAA_THIRD
Connections:
- removed net N$11: U$1.RA2, U$8.6
- removed net N$12: U$1.RC5, U$9.4
- removed net N$13: U$1.MCLR/VPP/RA3, U$8.1
- removed net N$14: U$1.RA0/ICSPDAT, U$8.4
- removed net N$15: U$1.RA1/ICSPCLK, U$8.5
- removed net N$17: U$1.RC4, U$9.3
- removed net N$18: U$1.RC2, U$9.1
- removed net N$20: U$2.B0, U$7.A
- removed net N$5: U$2.B1, U$4.4
- removed net N$8: U$3.B1, U$4.2
- removed net N$9: U$1.RA5, U$2.S, U$3.S
- net GND: now also R3.1, U$3.$2; no longer C1.2, C4.2, U$2.GND, U$3.GND, U$4.1, U$4.5, U$8.3
- net N$10: now also U$5.4; no longer U$5.2
- net N$2: now also U$2.$2, U$3.$1; no longer U$1.RC0, U$2.A
- net N$3: now also R3.2, TERMISTOR.2, U$1.RC2; no longer U$1.RC3, U$9.2
- net N$4: now also U$7.A; no longer U$3.A
- net N$6: now also U$5.2; no longer U$5.4
- net N$7: now also U$1.RC0; no longer U$3.B0
- net VCC: now also TERMISTOR.1, U$2.$1; no longer C1.1, C4.1, U$2.VCC, U$3.VCC, U$4.3, U$8.2
