File: Eagle/stavebnice03/misc/lipol_source.brd (EAGLE design)
At the start: 27 parts

Commit message: element position changed to be able put the bords to boxes + reset button for source board
Parts:
- removed U$4: JUMPER2M, !stavebnice03:JUMPER2M
- added U$6: BYTTON-B3U, !stavebnice03:BUTTON-B3U
- moved C6 1.14 mm to (12.7, 6.50), turned to 270 degrees
- moved C1 0.42 mm to (9.40, 11.4)
- moved U$9 0.32 mm to (12.6, 2.90)
- moved C4 0.20 mm to (8.50, 10.0)
- moved R4 0.10 mm to (5.80, 5.80)
- moved MCP73832 0.10 mm to (8.80, 7.50)
Connections:
- net GND: now also U$2.P$6, U$6.P$1, U$6.P$3; no longer U$2.P$4, U$4.2
- net N$20: now also U$6.P$2; no longer U$4.1
Routing:
- net N$20: track 4.05 -> 28.6 mm, vias 0 -> 1
- net GND: track 102.9 -> 109.1 mm
- net N$7: track 31.3 -> 27.2 mm
- net N$8: track 9.04 -> 9.99 mm
- net N$9: track 20.6 -> 19.6 mm
- net N$5: track 18.1 -> 17.3 mm
- net N$12: track 4.58 -> 4.01 mm
Other:
- board outline added: 21 x 21 mm
