File: Eagle/stavebnice03/base/action_module_base.sch (EAGLE design)
At the start: 9 parts

Commit message: layer coloring and place drawing moved to docu layer + changed sizes of names and values
Parts:
- renumbered U$1 to U1, U$2 to PROG, U$3 to DATA, U$4 to IN
Changed lines of the file:
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@@
 </classes>
 <parts>
-<part name="U$1" library="!stavebnice03" deviceset="16F103-TSSOP" device=""/>
+<part name="U1" library="!stavebnice03" deviceset="16F103-TSSOP" device=""/>
 <part name="C2" library="resistor" deviceset="C-EU" device="C0603K" value="100nF"/>
-<part name="U$4" library="!stavebnice03" deviceset="JUMPER5M-90" device=""/>
+<part name="IN" library="!stavebnice03" deviceset="JUMPER5M-90" device=""/>
 <part name="R3" library="resistor" deviceset="R-EU_" device="R0603" value="2K2"/>
 <part name="R4" library="resistor" deviceset="R-EU_" device="R0603" value="2k2"/>
 <part name="R1" library="resistor" deviceset="R-EU_" device="R0603" value="100k"/>
-<part name="U$2" library="!stavebnice03" deviceset="JUMPER5M" device=""/>
-<part name="U$3" library="!stavebnice03" deviceset="JUMPER5M" device=""/>
+<part name="PROG" library="!stavebnice03" deviceset="JUMPER5M" device=""/>
+<part name="DATA" library="!stavebnice03" deviceset="JUMPER5M" device=""/>
 <part name="TP1" library="testpad" deviceset="TP" device="B1,27"/>
 </parts>
@@
 </plain>
 <instances>
-<instance part="U$1" gate="G$1" x="144.78" y="86.36"/>
+<instance part="U1" gate="G$1" x="144.78" y="86.36"/>
 <instance part="C2" gate="G$1" x="144.78" y="104.14" rot="R90"/>
-<instance part="U$4" gate="G$1" x="91.44" y="165.1" rot="R180"/>
+<instance part="IN" gate="G$1" x="91.44" y="165.1" rot="R180"/>
 <instance part="R3" gate="G$1" x="106.68" y="144.78" rot="R270"/>
 <instance part="R4" gate="G$1" x="114.3" y="144.78" rot="R270"/>
 <instance part="R1" gate="G$1" x="109.22" y="93.98"/>
-<instance part="U$2" gate="G$1" x="172.72" y="35.56" rot="MR270"/>
-<instance part="U$3" gate="G$1" x="116.84" y="35.56" rot="R270"/>
+<instance part="PROG" gate="G$1" x="172.72" y="35.56" rot="MR270"/>
+<instance part="DATA" gate="G$1" x="116.84" y="35.56" rot="R270"/>
 <instance part="TP1" gate="G$1" x="116.84" y="101.6"/>
 </instances>
@@
 <wire x1="165.1" y1="154.94" x2="165.1" y2="175.26" width="0.1524" layer="91"/>
 <wire x1="165.1" y1="175.26" x2="99.06" y2="175.26" width="0.1524" layer="91"/>
-<pinref part="U$4" gate="G$1" pin="5"/>
-<pinref part="U$4" gate="G$1" pin="1"/>
+<pinref part="IN" gate="G$1" pin="5"/>
+<pinref part="IN" gate="G$1" pin="1"/>
 <wire x1="99.06" y1="154.94" x2="165.1" y2="154.94" width="0.1524" layer="91"/>
 <junction x="165.1" y="154.94"/>
@@
 <wire x1="172.72" y1="43.18" x2="172.72" y2="104.14" width="0.1524" layer="91"/>
 <wire x1="165.1" y1="104.14" x2="172.72" y2="104.14" width="0.1524" layer="91"/>
-<pinref part="U$1" gate="G$1" pin="GND"/>
+<pinref part="U1" gate="G$1" pin="GND"/>
 <wire x1="165.1" y1="99.06" x2="165.1" y2="104.14" width="0.1524" layer="91"/>
 <junction x="165.1" y="104.14"/>
 <pinref part="C2" gate="G$1" pin="2"/>
 <wire x1="149.86" y1="104.14" x2="165.1" y2="104.14" width="0.1524" layer="91"/>
-<pinref part="U$2" gate="G$1" pin="3"/>
+<pinref part="PROG" gate="G$1" pin="3"/>
 </segment>
 </net>
 <net name="VCC" class="0">
 <segment>
-<pinref part="U$1" gate="G$1" pin="VCC"/>
+<pinref part="U1" gate="G$1" pin="VCC"/>
 <wire x1="167.64" y1="109.22" x2="121.92" y2="109.22" width="0.1524" layer="91"/>
 <wire x1="121.92" y1="109.22" x2="114.3" y2="109.22" width="0.1524" layer="91"/>
@@
 <wire x1="142.24" y1="104.14" x2="121.92" y2="104.14" width="0.1524" layer="91"/>
 <junction x="121.92" y="104.14"/>
-<pinref part="U$4" gate="G$1" pin="3"/>
+<pinref part="IN" gate="G$1" pin="3"/>
 <pinref part="R4" gate="G$1" pin="2"/>
 <wire x1="114.3" y1="139.7" x2="114.3" y2="109.22" width="0.1524" layer="91"/>
@@
 <wire x1="101.6" y1="93.98" x2="101.6" y2="109.22" width="0.1524" layer="91"/>
 <wire x1="101.6" y1="109.22" x2="106.68" y2="109.22" width="0.1524" layer="91"/>
-<pinref part="U$2" gate="G$1" pin="2"/>
+<pinref part="PROG" gate="G$1" pin="2"/>
 <junction x="101.6" y="109.22"/>
 </segment>
@@
 <wire x1="162.56" y1="48.26" x2="101.6" y2="48.26" width="0.1524" layer="91"/>
 <wire x1="101.6" y1="48.26" x2="101.6" y2="83.82" width="0.1524" layer="91"/>
-<pinref part="U$1" gate="G$1" pin="MCLR/VPP/RA3"/>
+<pinref part="U1" gate="G$1" pin="MCLR/VPP/RA3"/>
 <wire x1="101.6" y1="83.82" x2="124.46" y2="83.82" width="0.1524" layer="91"/>
-<pinref part="U$2" gate="G$1" pin="1"/>
+<pinref part="PROG" gate="G$1" pin="1"/>
 </segment>
 </net>
@@
 <wire x1="177.8" y1="43.18" x2="177.8" y2="93.98" width="0.1524" layer="91"/>
 <wire x1="177.8" y1="93.98" x2="165.1" y2="93.98" width="0.1524" layer="91"/>
-<pinref part="U$1" gate="G$1" pin="RA0/ICSPDAT"/>
-<pinref part="U$2" gate="G$1" pin="4"/>
+<pinref part="U1" gate="G$1" pin="RA0/ICSPDAT"/>
+<pinref part="PROG" gate="G$1" pin="4"/>
 </segment>
 </net>
 <net name="N$15" class="0">
 <segment>
-<pinref part="U$1" gate="G$1" pin="RA1/ICSPCLK"/>
+<pinref part="U1" gate="G$1" pin="RA1/ICSPCLK"/>
 <wire x1="165.1" y1="88.9" x2="182.88" y2="88.9" width="0.1524" layer="91"/>
 <wire x1="182.88" y1="88.9" x2="182.88" y2="43.18" width="0.1524" layer="91"/>
-<pinref part="U$2" gate="G$1" pin="5"/>
+<pinref part="PROG" gate="G$1" pin="5"/>
 </segment>
 </net>
 <net name="N$11" class="0">
 <segment>
-<pinref part="U$1" gate="G$1" pin="RA2"/>
+<pinref part="U1" gate="G$1" pin="RA2"/>
 <wire x1="165.1" y1="83.82" x2="187.96" y2="83.82" width="0.1524" layer="91"/>
 <wire x1="187.96" y1="83.82" x2="187.96" y2="58.42" width="0.1524" layer="91"/>
 <wire x1="187.96" y1="58.42" x2="106.68" y2="58.42" width="0.1524" layer="91"/>
 <wire x1="106.68" y1="58.42" x2="106.68" y2="43.18" width="0.1524" layer="91"/>
-<pinref part="U$3" gate="G$1" pin="5"/>
+<pinref part="DATA" gate="G$1" pin="5"/>
 </segment>
 </net>
 <net name="N$18" class="0">
 <segment>
-<pinref part="U$1" gate="G$1" pin="RC2"/>
+<pinref part="U1" gate="G$1" pin="RC2"/>
 <wire x1="165.1" y1="53.34" x2="165.1" y2="68.58" width="0.1524" layer="91"/>
 <wire x1="165.1" y1="53.34" x2="127" y2="53.34" width="0.1524" layer="91"/>
 <wire x1="127" y1="53.34" x2="127" y2="43.18" width="0.1524" layer="91"/>
-<pinref part="U$3" gate="G$1" pin="1"/>
+<pinref part="DATA" gate="G$1" pin="1"/>
 </segment>
 </net>
 <net name="N$17" class="0">
 <segment>
-<pinref part="U$1" gate="G$1" pin="RC4"/>
+<pinref part="U1" gate="G$1" pin="RC4"/>
 <wire x1="124.46" y1="73.66" x2="116.84" y2="73.66" width="0.1524" layer="91"/>
 <wire x1="116.84" y1="73.66" x2="116.84" y2="43.18" width="0.1524" layer="91"/>
-<pinref part="U$3" gate="G$1" pin="3"/>
+<pinref part="DATA" gate="G$1" pin="3"/>
 </segment>
 </net>
 <net name="N$12" class="0">
 <segment>
-<pinref part="U$1" gate="G$1" pin="RC5"/>
+<pinref part="U1" gate="G$1" pin="RC5"/>
 <wire x1="124.46" y1="78.74" x2="111.76" y2="78.74" width="0.1524" layer="91"/>
 <wire x1="111.76" y1="78.74" x2="111.76" y2="43.18" width="0.1524" layer="91"/>
-<pinref part="U$3" gate="G$1" pin="4"/>
+<pinref part="DATA" gate="G$1" pin="4"/>
 </segment>
 </net>
 <net name="N$5" class="0">
 <segment>
-<pinref part="U$4" gate="G$1" pin="4"/>
+<pinref part="IN" gate="G$1" pin="4"/>
 <wire x1="99.06" y1="170.18" x2="114.3" y2="170.18" width="0.1524" layer="91"/>
 <wire x1="114.3" y1="170.18" x2="195.58" y2="170.18" width="0.1524" layer="91"/>
 <wire x1="195.58" y1="170.18" x2="195.58" y2="73.66" width="0.1524" layer="91"/>
-<pinref part="U$1" gate="G$1" pin="RC1"/>
+<pinref part="U1" gate="G$1" pin="RC1"/>
 <wire x1="165.1" y1="73.66" x2="195.58" y2="73.66" width="0.1524" layer="91"/>
 <pinref part="R4" gate="G$1" pin="1"/>
@@
 <net name="N$2" class="0">
 <segment>
-<pinref part="U$1" gate="G$1" pin="RC0"/>
+<pinref part="U1" gate="G$1" pin="RC0"/>
 <wire x1="190.5" y1="78.74" x2="165.1" y2="78.74" width="0.1524" layer="91"/>
-<pinref part="U$4" gate="G$1" pin="2"/>
+<pinref part="IN" gate="G$1" pin="2"/>
 <wire x1="190.5" y1="78.74" x2="190.5" y2="160.02" width="0.1524" layer="91"/>
 <wire x1="190.5" y1="160.02" x2="106.68" y2="160.02" width="0.1524" layer="91"/>
@@
 <net name="N$1" class="0">
 <segment>
-<pinref part="U$1" gate="G$1" pin="RC3"/>
+<pinref part="U1" gate="G$1" pin="RC3"/>
 <wire x1="121.92" y1="43.18" x2="121.92" y2="68.58" width="0.1524" layer="91"/>
 <wire x1="121.92" y1="68.58" x2="124.46" y2="68.58" width="0.1524" layer="91"/>
-<pinref part="U$3" gate="G$1" pin="2"/>
+<pinref part="DATA" gate="G$1" pin="2"/>
 </segment>
 </net>
 <net name="N$3" class="0">
 <segment>
-<pinref part="U$1" gate="G$1" pin="RA5"/>
+<pinref part="U1" gate="G$1" pin="RA5"/>
 <pinref part="R1" gate="G$1" pin="2"/>
 <wire x1="124.46" y1="93.98" x2="116.84" y2="93.98" width="0.1524" layer="91"/>

Commit message: eagle adjustment for the Jíťa version
Parts:
- renumbered TP1 to FLASH
Changed lines of the file:
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@@
 <part name="R4" library="resistor" deviceset="R-EU_" device="R0603" value="2k2"/>
 <part name="R1" library="resistor" deviceset="R-EU_" device="R0603" value="100k"/>
-<part name="PROG" library="!stavebnice03" deviceset="JUMPER5M" device=""/>
-<part name="DATA" library="!stavebnice03" deviceset="JUMPER5M" device=""/>
-<part name="TP1" library="testpad" deviceset="TP" device="B1,27"/>
+<part name="PROG" library="!stavebnice03" deviceset="JUMPER5M" device="" value=""/>
+<part name="DATA" library="!stavebnice03" deviceset="JUMPER5M" device="" value=""/>
+<part name="FLASH" library="testpad" deviceset="TP" device="B1,27"/>
 </parts>
 <sheets>
@@
 <instance part="PROG" gate="G$1" x="172.72" y="35.56" rot="MR270"/>
 <instance part="DATA" gate="G$1" x="116.84" y="35.56" rot="R270"/>
-<instance part="TP1" gate="G$1" x="116.84" y="101.6"/>
+<instance part="FLASH" gate="G$1" x="116.84" y="101.6"/>
 </instances>
 <busses>
@@
 <pinref part="R1" gate="G$1" pin="2"/>
 <wire x1="124.46" y1="93.98" x2="116.84" y2="93.98" width="0.1524" layer="91"/>
-<pinref part="TP1" gate="G$1" pin="TP"/>
+<pinref part="FLASH" gate="G$1" pin="TP"/>
 <wire x1="116.84" y1="93.98" x2="114.3" y2="93.98" width="0.1524" layer="91"/>
 <wire x1="116.84" y1="99.06" x2="116.84" y2="93.98" width="0.1524" layer="91"/>
