File: Eagle/manabu/base/action_module_base.sch (EAGLE design)
At the start: 9 parts, among them U1 16F103-TSSOP

Commit message: preparation for the seed studio PCB maker
Parts:
- C2: value 100nF -> 100n
- FLASH: value TPB1,27 -> TPTP10R; device testpad:TPB1,27 -> testpad:TPTP10R
- U1: value 16F103-TSSOP -> 16F103
Changed lines of the file:
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@@
 </classes>
 <parts>
-<part name="U1" library="!stavebnice03" deviceset="16F103-TSSOP" device=""/>
-<part name="C2" library="resistor" deviceset="C-EU" device="C0603K" value="100nF"/>
+<part name="U1" library="!stavebnice03" deviceset="16F103-TSSOP" device="" value="16F103"/>
+<part name="C2" library="resistor" deviceset="C-EU" device="C0603K" value="100n"/>
 <part name="IN" library="!stavebnice03" deviceset="JUMPER5M-90" device=""/>
 <part name="R3" library="resistor" deviceset="R-EU_" device="R0603" value="2K2"/>
 <part name="R4" library="resistor" deviceset="R-EU_" device="R0603" value="2k2"/>
 <part name="R1" library="resistor" deviceset="R-EU_" device="R0603" value="100k"/>
-<part name="PROG" library="!stavebnice03" deviceset="JUMPER5M" device="" value=""/>
-<part name="DATA" library="!stavebnice03" deviceset="JUMPER5M" device="" value=""/>
-<part name="FLASH" library="testpad" deviceset="TP" device="B1,27"/>
+<part name="PROG" library="!stavebnice03" deviceset="JUMPER5M" device="" value="JUMPER5M"/>
+<part name="DATA" library="!stavebnice03" deviceset="JUMPER5M" device="" value="JUMPER5M"/>
+<part name="FLASH" library="testpad" deviceset="TP" device="TP10R" value="TPTP10R"/>
 </parts>
 <sheets>
