File: Eagle/manabu/base/sensor_module_base.brd (EAGLE design)
At the start: 21 x 21 mm, 19 parts, among them U1 16F103, U2 NC7SB3157P6X, U3 NC7SB3157P6X, U4 NC7SB3157P6X, U5 NC7SB3157P6X

Commit message: just a few optimalization on the sensor board
Parts:
- R3: value 2K2 -> 2k2
- U1: value 16F103 -> 16F1503
- moved R3 1.14 mm to (11.3, 13.6), turned to 90 degrees
- moved R1 0.72 mm to (15.0, 13.6)
- moved R4 0.22 mm to (11.3, 9.50)
- moved C5 0.10 mm to (15.2, 14.4)
Routing:
- net N$14: track 7.87 -> 5.14 mm
- net VCC: track 55.7 -> 58.4 mm
- net N$13: track 18.3 -> 17.3 mm
- net GND: track 78.0 -> 78.8 mm, vias 3 -> 2
- net N$8: track 7.81 -> 8.45 mm
- net N$1: track 24.8 -> 25.4 mm
- removed copper zone on layer 1, net N$2
- removed copper zone on layer 16, net N$20
Other:
- board text added: "sensor v0.2"
- board text removed: "sensor v0.1"
