File: Eagle/manabu/base/sensor_module_base.sch (EAGLE design)
At the start: 19 parts, among them U1 16F103, U2 NC7SB3157P6X, U3 NC7SB3157P6X, U4 NC7SB3157P6X, U5 NC7SB3157P6X

Commit message: just a few optimalization on the sensor board
Parts:
- R3: value 2K2 -> 2k2
- U1: value 16F103 -> 16F1503
Changed lines of the file:
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@@
 <?xml version="1.0" encoding="utf-8"?>
 <!DOCTYPE eagle SYSTEM "eagle.dtd">
-<eagle version="7.2.0">
+<eagle version="7.4.0">
 <drawing>
 <settings>
@@
 </classes>
 <parts>
-<part name="U1" library="!stavebnice03" deviceset="16F103-TSSOP" device="" value="16F103"/>
+<part name="U1" library="!stavebnice03" deviceset="16F103-TSSOP" device="" value="16F1503"/>
 <part name="C2" library="resistor" deviceset="C-EU" device="C0603K" value="100n"/>
 <part name="R1" library="resistor" deviceset="R-EU_" device="R0603" value="2k2"/>
@@
 <part name="C4" library="resistor" deviceset="C-EU" device="C0603K" value="100n"/>
 <part name="DATA" library="!stavebnice03" deviceset="JUMPER4M" device="" value="JUMPER4M"/>
-<part name="R3" library="resistor" deviceset="R-EU_" device="R0603" value="2K2"/>
+<part name="R3" library="resistor" deviceset="R-EU_" device="R0603" value="2k2"/>
 <part name="R4" library="resistor" deviceset="R-EU_" device="R0603" value="2k2"/>
 <part name="R5" library="resistor" deviceset="R-EU_" device="R0603" value="100k"/>
@@
 <wire x1="101.6" y1="58.42" x2="101.6" y2="88.9" width="0.1524" layer="91"/>
 <pinref part="U1" gate="G$1" pin="RA4"/>
+<pinref part="U5" gate="G$1" pin="S"/>
 <wire x1="101.6" y1="88.9" x2="124.46" y2="88.9" width="0.1524" layer="91"/>
-<pinref part="U5" gate="G$1" pin="S"/>
 <wire x1="238.76" y1="73.66" x2="246.38" y2="73.66" width="0.1524" layer="91"/>
 <pinref part="U4" gate="G$1" pin="S"/>
