File: Eagle/manabu/misc/lipol_source.brd (EAGLE design)
At the start: 21 x 21 mm, 29 parts, among them T1 FDV304P, U1 16F1454, U2 NC7SB3157P6X, U3 NC7SB3157P6X

Commit message: invert output functionality moved to lipol module port A4 to be as same as on other modules (bootloader reset pin will have to be changed for lipol module)
Parts:
- R2: value 2k2 -> 2_k2
Connections:
- net N$1: now also U1.3; no longer U1.2
Routing:
- net N$1: track 12.9 -> 13.6 mm
Other:
- board text added: "LiPol v0.2"
- board text removed: "LiPol v0.1"
